File: laptop_kbrd.sch (KiCad schematic (older format))
At the start: 62 parts, among them CON1 AVR-ISP-6-DR, K1 CASE_OPEN, Q1 MOSFET_N, Q2 MOSFET_N, Q3 MOSFET_N, Q4 MOSFET_N, Q5 MOSFET_N, Q6 MOSFET_N, Q7 MOSFET_N, Q8 ALS_PT19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

Commit message: We'll need to do something about track clearances in PCB.
Changed lines of the file:
@@
 Sheet 1 1
 Title ""
-Date "10 nov 2015"
+Date "14 nov 2015"
 Rev ""
 Comp ""
@@
 L GND #PWR06
 U 1 1 563D8E9D
-P 7200 3450
-F 0 "#PWR06" H 7200 3450 30  0001 C CNN
-F 1 "GND" H 7200 3380 30  0001 C CNN
-F 2 "" H 7200 3450 60  0000 C CNN
-F 3 "" H 7200 3450 60  0000 C CNN
-	1    7200 3450
+P 7200 3500
+F 0 "#PWR06" H 7200 3500 30  0001 C CNN
+F 1 "GND" H 7200 3430 30  0001 C CNN
+F 2 "" H 7200 3500 60  0000 C CNN
+F 3 "" H 7200 3500 60  0000 C CNN
+	1    7200 3500
 	1    0    0    -1
 $EndComp
@@
 	5300 3200 5300 3300
 Wire Wire Line
-	7300 3350 7200 3350
-Wire Wire Line
-	7200 3350 7200 3450
-Wire Wire Line
 	9200 3200 9100 3200
 Wire Wire Line
@@
 Wire Wire Line
 	9200 3200 9200 3850
-Wire Wire Line
-	7300 3350 7300 4100
 Wire Wire Line
 	5400 3200 5400 3850
@@
 Connection ~ 8500 4950
 Connection ~ 7800 4950
+Wire Wire Line
+	7200 3500 7200 3450
+Wire Wire Line
+	7200 3450 7300 3450
+Wire Wire Line
+	7300 3450 7300 4100
 $EndSCHEMATC

Commit message: Removed RCLAMP
Parts:
- removed U3: RCLAMP0502B, symbol RCLAMP0502B
Connections:
- wire segments 324 -> 323
Changed lines of the file:
@@
 Sheet 1 1
 Title ""
-Date "14 nov 2015"
+Date "17 nov 2015"
 Rev ""
 Comp ""
@@
 Connection ~ 1000 4250
 Wire Wire Line
-	8500 5350 10200 5350
-Wire Wire Line
 	10200 5250 9450 5250
 Wire Wire Line
@@
 Connection ~ 9450 6550
 $Comp
-L RCLAMP0502B U3
-U 1 1 56403FC5
-P 8100 6450
-F 0 "U3" V 8450 6450 60  0000 C CNN
-F 1 "RCLAMP0502B" V 7800 6400 60  0000 C CNN
-F 2 "" H 8100 6450 60  0000 C CNN
-F 3 "" H 8100 6450 60  0000 C CNN
-	1    8100 6450
-	0    -1   -1   0
-$EndComp
-$Comp
-L GND #PWR027
-U 1 1 56403FE1
-P 8700 6600
-F 0 "#PWR027" H 8700 6600 30  0001 C CNN
-F 1 "GND" H 8700 6530 30  0001 C CNN
-F 2 "" H 8700 6600 60  0000 C CNN
-F 3 "" H 8700 6600 60  0000 C CNN
-	1    8700 6600
-	1    0    0    -1
-$EndComp
-Wire Wire Line
-	8600 6450 8700 6450
-Wire Wire Line
-	8700 6450 8700 6600
-Wire Wire Line
-	7650 6300 7250 6300
-Wire Wire Line
-	7650 6600 7250 6600
-Text Label 7250 6300 0    60   ~ 0
-D+
-Text Label 7250 6600 0    60   ~ 0
-D-
-$Comp
 L C C8
 U 1 1 56417885
@@
 Wire Wire Line
 	7300 3450 7300 4100
+Wire Wire Line
+	8650 5350 8650 5150
+Wire Wire Line
+	8650 5150 7900 5150
+Wire Wire Line
+	7900 5150 7900 5350
+Wire Wire Line
+	8650 5350 10200 5350
 $EndSCHEMATC

Commit message: Added lidsense. Mounting holes.
Parts:
- added K2: CASE_OPEN, ~, symbol CONN_3
- added R23: 47K, ~, symbol R
- added SW4: CASE_PUSH, ~, symbol DPST_SMALL
Connections:
- wire segments 323 -> 329
Changed lines of the file:
@@
 Sheet 1 1
 Title ""
-Date "17 nov 2015"
+Date "19 nov 2015"
 Rev ""
 Comp ""
@@
 $EndComp
 $Comp
-L VCC #PWR01
+L VCC #PWR2
 U 1 1 563D8577
 P 1750 950
-F 0 "#PWR01" H 1750 1050 30  0001 C CNN
+F 0 "#PWR2" H 1750 1050 30  0001 C CNN
 F 1 "VCC" H 1750 1050 30  0000 C CNN
 F 2 "" H 1750 950 60  0000 C CNN
@@
 $EndComp
 $Comp
-L GND #PWR02
+L GND #PWR3
 U 1 1 563D875C
 P 1750 4450
-F 0 "#PWR02" H 1750 4450 30  0001 C CNN
+F 0 "#PWR3" H 1750 4450 30  0001 C CNN
 F 1 "GND" H 1750 4380 30  0001 C CNN
 F 2 "" H 1750 4450 60  0000 C CNN
@@
 $EndComp
 $Comp
-L VDD #PWR03
+L VDD #PWR26
 U 1 1 563D8C10
 P 10850 1250
-F 0 "#PWR03" H 10850 1350 30  0001 C CNN
+F 0 "#PWR26" H 10850 1350 30  0001 C CNN
 F 1 "VDD" H 10850 1360 30  0000 C CNN
 F 2 "" H 10850 1250 60  0000 C CNN
@@
 $EndComp
 $Comp
-L VDD #PWR04
+L VDD #PWR15
 U 1 1 563D8C1D
 P 6700 1300
-F 0 "#PWR04" H 6700 1400 30  0001 C CNN
+F 0 "#PWR15" H 6700 1400 30  0001 C CNN
 F 1 "VDD" H 6700 1410 30  0000 C CNN
 F 2 "" H 6700 1300 60  0000 C CNN
@@
 $EndComp
 $Comp
-L GND #PWR05
+L GND #PWR8
 U 1 1 563D8E97
 P 5300 3300
-F 0 "#PWR05" H 5300 3300 30  0001 C CNN
+F 0 "#PWR8" H 5300 3300 30  0001 C CNN
 F 1 "GND" H 5300 3230 30  0001 C CNN
 F 2 "" H 5300 3300 60  0000 C CNN
@@
 $EndComp
 $Comp
-L GND #PWR06
+L GND #PWR17
 U 1 1 563D8E9D
 P 7200 3500
-F 0 "#PWR06" H 7200 3500 30  0001 C CNN
+F 0 "#PWR17" H 7200 3500 30  0001 C CNN
 F 1 "GND" H 7200 3430 30  0001 C CNN
 F 2 "" H 7200 3500 60  0000 C CNN
@@
 $EndComp
 $Comp
-L GND #PWR07
+L GND #PWR21
 U 1 1 563D8EA3
 P 9100 3300
-F 0 "#PWR07" H 9100 3300 30  0001 C CNN
+F 0 "#PWR21" H 9100 3300 30  0001 C CNN
 F 1 "GND" H 9100 3230 30  0001 C CNN
 F 2 "" H 9100 3300 60  0000 C CNN
@@
 $EndComp
 $Comp
-L GND #PWR08
+L GND #PWR25
 U 1 1 563D8EA9
 P 10850 900
-F 0 "#PWR08" H 10850 900 30  0001 C CNN
+F 0 "#PWR25" H 10850 900 30  0001 C CNN
 F 1 "GND" H 10850 830 30  0001 C CNN
 F 2 "" H 10850 900 60  0000 C CNN
@@
 $EndComp
 $Comp
-L GND #PWR09
+L GND #PWR14
 U 1 1 563D8EAF
 P 6700 900
-F 0 "#PWR09" H 6700 900 30  0001 C CNN
+F 0 "#PWR14" H 6700 900 30  0001 C CNN
 F 1 "GND" H 6700 830 30  0001 C CNN
 F 2 "" H 6700 900 60  0000 C CNN
@@
 $EndComp
 $Comp
-L VCC #PWR010
+L VCC #PWR7
 U 1 1 563D935F
 P 5300 3000
-F 0 "#PWR010" H 5300 3100 30  0001 C CNN
+F 0 "#PWR7" H 5300 3100 30  0001 C CNN
 F 1 "VCC" H 5300 3100 30  0000 C CNN
 F 2 "" H 5300 3000 60  0000 C CNN
@@
 $EndComp
 $Comp
-L VCC #PWR011
+L VCC #PWR16
 U 1 1 563D9365
 P 7200 3250
-F 0 "#PWR011" H 7200 3350 30  0001 C CNN
+F 0 "#PWR16" H 7200 3350 30  0001 C CNN
 F 1 "VCC" H 7200 3350 30  0000 C CNN
 F 2 "" H 7200 3250 60  0000 C CNN
@@
 $EndComp
 $Comp
-L VCC #PWR012
+L VCC #PWR20
 U 1 1 563D936B
 P 9100 3000
-F 0 "#PWR012" H 9100 3100 30  0001 C CNN
+F 0 "#PWR20" H 9100 3100 30  0001 C CNN
 F 1 "VCC" H 9100 3100 30  0000 C CNN
 F 2 "" H 9100 3000 60  0000 C CNN
@@
 $EndComp
 $Comp
-L VDD #PWR013
+L VDD #PWR12
 U 1 1 563E23A9
 P 5850 7300
-F 0 "#PWR013" H 5850 7400 30  0001 C CNN
+F 0 "#PWR12" H 5850 7400 30  0001 C CNN
 F 1 "VDD" H 5850 7410 30  0000 C CNN
 F 2 "" H 5850 7300 60  0000 C CNN
@@
 5V_DELAYED
 $Comp
-L VCC #PWR014
+L VCC #PWR22
 U 1 1 563E27AB
 P 9450 6450
-F 0 "#PWR014" H 9450 6550 30  0001 C CNN
+F 0 "#PWR22" H 9450 6550 30  0001 C CNN
 F 1 "VCC" H 9450 6550 30  0000 C CNN
 F 2 "" H 9450 6450 60  0000 C CNN
@@
 $EndComp
 $Comp
-L GND #PWR015
+L GND #PWR23
 U 1 1 563E2834
 P 10050 7100
-F 0 "#PWR015" H 10050 7100 30  0001 C CNN
+F 0 "#PWR23" H 10050 7100 30  0001 C CNN
 F 1 "GND" H 10050 7030 30  0001 C CNN
 F 2 "" H 10050 7100 60  0000 C CNN
@@
 D-
 $Comp
-L GND #PWR016
+L GND #PWR1
 U 1 1 563E311C
 P 850 7700
-F 0 "#PWR016" H 850 7700 30  0001 C CNN
+F 0 "#PWR1" H 850 7700 30  0001 C CNN
 F 1 "GND" H 850 7630 30  0001 C CNN
 F 2 "" H 850 7700 60  0000 C CNN
@@
 $EndComp
 $Comp
-L GND #PWR017
+L GND #PWR11
 U 1 1 563ED260
 P 5400 1000
-F 0 "#PWR017" H 5400 1000 30  0001 C CNN
+F 0 "#PWR11" H 5400 1000 30  0001 C CNN
 F 1 "GND" H 5400 930 30  0001 C CNN
 F 2 "" H 5400 1000 60  0000 C CNN
@@
 MISO
 $Comp
-L VCC #PWR018
+L VCC #PWR10
 U 1 1 563EDBAF
 P 5400 700
-F 0 "#PWR018" H 5400 800 30  0001 C CNN
+F 0 "#PWR10" H 5400 800 30  0001 C CNN
 F 1 "VCC" H 5400 800 30  0000 C CNN
 F 2 "" H 5400 700 60  0000 C CNN
@@
 $EndComp
 $Comp
-L GND #PWR019
+L GND #PWR9
 U 1 1 563EFB35
 P 5350 2150
-F 0 "#PWR019" H 5350 2150 30  0001 C CNN
+F 0 "#PWR9" H 5350 2150 30  0001 C CNN
 F 1 "GND" H 5350 2080 30  0001 C CNN
 F 2 "" H 5350 2150 60  0000 C CNN
@@
 $EndComp
 $Comp
-L GND #PWR020
+L GND #PWR24
 U 1 1 563F09B8
 P 10750 2450
-F 0 "#PWR020" H 10750 2450 30  0001 C CNN
+F 0 "#PWR24" H 10750 2450 30  0001 C CNN
 F 1 "GND" H 10750 2380 30  0001 C CNN
 F 2 "" H 10750 2450 60  0000 C CNN
@@
 $EndComp
 $Comp
-L GND #PWR021
+L GND #PWR19
 U 1 1 563F123A
 P 8700 5600
-F 0 "#PWR021" H 8700 5600 30  0001 C CNN
+F 0 "#PWR19" H 8700 5600 30  0001 C CNN
 F 1 "GND" H 8700 5530 30  0001 C CNN
 F 2 "" H 8700 5600 60  0000 C CNN
@@
 $EndComp
 $Comp
-L GND #PWR022
+L GND #PWR18
 U 1 1 563F1826
 P 7800 5050
-F 0 "#PWR022" H 7800 5050 30  0001 C CNN
+F 0 "#PWR18" H 7800 5050 30  0001 C CNN
 F 1 "GND" H 7800 4980 30  0001 C CNN
 F 2 "" H 7800 5050 60  0000 C CNN
@@
 $EndComp
 $Comp
-L VDD #PWR023
+L VDD #PWR5
 U 1 1 563EF135
 P 3250 5000
-F 0 "#PWR023" H 3250 5100 30  0001 C CNN
+F 0 "#PWR5" H 3250 5100 30  0001 C CNN
 F 1 "VDD" H 3250 5110 30  0000 C CNN
 F 2 "" H 3250 5000 60  0000 C CNN
@@
 $EndComp
 $Comp
-L GND #PWR024
+L GND #PWR4
 U 1 1 563F26E5
 P 3000 6950
-F 0 "#PWR024" H 3000 6950 30  0001 C CNN
+F 0 "#PWR4" H 3000 6950 30  0001 C CNN
 F 1 "GND" H 3000 6880 30  0001 C CNN
 F 2 "" H 3000 6950 60  0000 C CNN
@@
 $EndComp
 $Comp
-L GND #PWR025
+L GND #PWR6
 U 1 1 5640122A
 P 3950 7700
-F 0 "#PWR025" H 3950 7700 30  0001 C CNN
+F 0 "#PWR6" H 3950 7700 30  0001 C CNN
 F 1 "GND" H 3950 7630 30  0001 C CNN
 F 2 "" H 3950 7700 60  0000 C CNN
@@
 $EndComp
 $Comp
-L GND #PWR026
+L GND #PWR13
 U 1 1 56401BCE
 P 6600 7350
-F 0 "#PWR026" H 6600 7350 30  0001 C CNN
+F 0 "#PWR13" H 6600 7350 30  0001 C CNN
 F 1 "GND" H 6600 7280 30  0001 C CNN
 F 2 "" H 6600 7350 60  0000 C CNN
@@
 Wire Wire Line
 	8650 5350 10200 5350
+$Comp
+L CONN_3 K2
+U 1 1 564D4485
+P 8850 6200
+F 0 "K2" V 8800 6200 50  0000 C CNN
+F 1 "CASE_OPEN" H 9050 6000 40  0000 C CNN
+F 2 "~" H 8850 6200 60  0000 C CNN
+F 3 "~" H 8850 6200 60  0000 C CNN
+	1    8850 6200
+	1    0    0    -1
+$EndComp
+$Comp
+L DPST_SMALL SW4
+U 1 1 564D448B
+P 7950 6200
+F 0 "SW4" H 7950 6000 70  0000 C CNN
+F 1 "CASE_PUSH" H 7950 6450 70  0000 C CNN
+F 2 "~" H 7950 6200 60  0000 C CNN
+F 3 "~" H 7950 6200 60  0000 C CNN
+	1    7950 6200
+	1    0    0    -1
+$EndComp
+$Comp
+L R R23
+U 1 1 564D4496
+P 8400 6450
+F 0 "R23" V 8480 6450 40  0000 C CNN
+F 1 "47K" V 8407 6451 40  0000 C CNN
+F 2 "~" V 8330 6450 30  0000 C CNN
+F 3 "~" H 8400 6450 30  0000 C CNN
+	1    8400 6450
+	-1   0    0    1
+$EndComp
+Wire Wire Line
+	8300 6200 8500 6200
+Wire Wire Line
+	8500 6300 8500 6700
+Wire Wire Line
+	8500 6700 8400 6700
+Wire Wire Line
+	8250 6300 8300 6300
+Wire Wire Line
+	8300 6300 8300 6200
+Connection ~ 8400 6200
+Wire Wire Line
+	8250 6100 8500 6100
 $EndSCHEMATC

Commit message: New components for the LCD controller.
Parts:
- added R24: 10K, ~, symbol R
Connections:
- wire segments 329 -> 333
- no-connect marks 15 -> 14
Changed lines of the file:
@@
 $Descr A4 11693 8268
 encoding utf-8
-Sheet 1 1
+Sheet 1 2
 Title ""
-Date "19 nov 2015"
+Date "3 mar 2016"
 Rev ""
 Comp ""
@@
 $EndComp
 $Comp
-L VCC #PWR2
+L VCC #PWR01
 U 1 1 563D8577
 P 1750 950
-F 0 "#PWR2" H 1750 1050 30  0001 C CNN
+F 0 "#PWR01" H 1750 1050 30  0001 C CNN
 F 1 "VCC" H 1750 1050 30  0000 C CNN
 F 2 "" H 1750 950 60  0000 C CNN
@@
 $EndComp
 $Comp
-L GND #PWR3
+L GND #PWR02
 U 1 1 563D875C
 P 1750 4450
-F 0 "#PWR3" H 1750 4450 30  0001 C CNN
+F 0 "#PWR02" H 1750 4450 30  0001 C CNN
 F 1 "GND" H 1750 4380 30  0001 C CNN
 F 2 "" H 1750 4450 60  0000 C CNN
@@
 $EndComp
 $Comp
-L VDD #PWR26
+L VDD #PWR03
 U 1 1 563D8C10
 P 10850 1250
-F 0 "#PWR26" H 10850 1350 30  0001 C CNN
+F 0 "#PWR03" H 10850 1350 30  0001 C CNN
 F 1 "VDD" H 10850 1360 30  0000 C CNN
 F 2 "" H 10850 1250 60  0000 C CNN
@@
 $EndComp
 $Comp
-L VDD #PWR15
+L VDD #PWR04
 U 1 1 563D8C1D
 P 6700 1300
-F 0 "#PWR15" H 6700 1400 30  0001 C CNN
+F 0 "#PWR04" H 6700 1400 30  0001 C CNN
 F 1 "VDD" H 6700 1410 30  0000 C CNN
 F 2 "" H 6700 1300 60  0000 C CNN
@@
 $EndComp
 $Comp
-L GND #PWR8
+L GND #PWR05
 U 1 1 563D8E97
 P 5300 3300
-F 0 "#PWR8" H 5300 3300 30  0001 C CNN
+F 0 "#PWR05" H 5300 3300 30  0001 C CNN
 F 1 "GND" H 5300 3230 30  0001 C CNN
 F 2 "" H 5300 3300 60  0000 C CNN
@@
 $EndComp
 $Comp
-L GND #PWR17
+L GND #PWR06
 U 1 1 563D8E9D
 P 7200 3500
-F 0 "#PWR17" H 7200 3500 30  0001 C CNN
+F 0 "#PWR06" H 7200 3500 30  0001 C CNN
 F 1 "GND" H 7200 3430 30  0001 C CNN
 F 2 "" H 7200 3500 60  0000 C CNN
@@
 $EndComp
 $Comp
-L GND #PWR21
+L GND #PWR07
 U 1 1 563D8EA3
 P 9100 3300
-F 0 "#PWR21" H 9100 3300 30  0001 C CNN
+F 0 "#PWR07" H 9100 3300 30  0001 C CNN
 F 1 "GND" H 9100 3230 30  0001 C CNN
 F 2 "" H 9100 3300 60  0000 C CNN
@@
 $EndComp
 $Comp
-L GND #PWR25
+L GND #PWR08
 U 1 1 563D8EA9
 P 10850 900
-F 0 "#PWR25" H 10850 900 30  0001 C CNN
+F 0 "#PWR08" H 10850 900 30  0001 C CNN
 F 1 "GND" H 10850 830 30  0001 C CNN
 F 2 "" H 10850 900 60  0000 C CNN
@@
 $EndComp
 $Comp
-L GND #PWR14
+L GND #PWR09
 U 1 1 563D8EAF
 P 6700 900
-F 0 "#PWR14" H 6700 900 30  0001 C CNN
+F 0 "#PWR09" H 6700 900 30  0001 C CNN
 F 1 "GND" H 6700 830 30  0001 C CNN
 F 2 "" H 6700 900 60  0000 C CNN
@@
 $EndComp
 $Comp
-L VCC #PWR7
+L VCC #PWR010
 U 1 1 563D935F
 P 5300 3000
-F 0 "#PWR7" H 5300 3100 30  0001 C CNN
+F 0 "#PWR010" H 5300 3100 30  0001 C CNN
 F 1 "VCC" H 5300 3100 30  0000 C CNN
 F 2 "" H 5300 3000 60  0000 C CNN
@@
 $EndComp
 $Comp
-L VCC #PWR16
+L VCC #PWR011
 U 1 1 563D9365
 P 7200 3250
-F 0 "#PWR16" H 7200 3350 30  0001 C CNN
+F 0 "#PWR011" H 7200 3350 30  0001 C CNN
 F 1 "VCC" H 7200 3350 30  0000 C CNN
 F 2 "" H 7200 3250 60  0000 C CNN
@@
 $EndComp
 $Comp
-L VCC #PWR20
+L VCC #PWR012
 U 1 1 563D936B
 P 9100 3000
-F 0 "#PWR20" H 9100 3100 30  0001 C CNN
+F 0 "#PWR012" H 9100 3100 30  0001 C CNN
 F 1 "VCC" H 9100 3100 30  0000 C CNN
 F 2 "" H 9100 3000 60  0000 C CNN
@@
 $EndComp
 $Comp
-L VDD #PWR12
+L VDD #PWR013
 U 1 1 563E23A9
 P 5850 7300
-F 0 "#PWR12" H 5850 7400 30  0001 C CNN
+F 0 "#PWR013" H 5850 7400 30  0001 C CNN
 F 1 "VDD" H 5850 7410 30  0000 C CNN
 F 2 "" H 5850 7300 60  0000 C CNN
@@
 5V_DELAYED
 $Comp
-L VCC #PWR22
+L VCC #PWR014
 U 1 1 563E27AB
 P 9450 6450
-F 0 "#PWR22" H 9450 6550 30  0001 C CNN
+F 0 "#PWR014" H 9450 6550 30  0001 C CNN
 F 1 "VCC" H 9450 6550 30  0000 C CNN
 F 2 "" H 9450 6450 60  0000 C CNN
@@
 $EndComp
 $Comp
-L GND #PWR23
+L GND #PWR015
 U 1 1 563E2834
 P 10050 7100
-F 0 "#PWR23" H 10050 7100 30  0001 C CNN
+F 0 "#PWR015" H 10050 7100 30  0001 C CNN
 F 1 "GND" H 10050 7030 30  0001 C CNN
 F 2 "" H 10050 7100 60  0000 C CNN
@@
 D-
 $Comp
-L GND #PWR1
+L GND #PWR016
 U 1 1 563E311C
 P 850 7700
-F 0 "#PWR1" H 850 7700 30  0001 C CNN
+F 0 "#PWR016" H 850 7700 30  0001 C CNN
 F 1 "GND" H 850 7630 30  0001 C CNN
 F 2 "" H 850 7700 60  0000 C CNN
@@
 $EndComp
 $Comp
-L GND #PWR11
+L GND #PWR017
 U 1 1 563ED260
 P 5400 1000
-F 0 "#PWR11" H 5400 1000 30  0001 C CNN
+F 0 "#PWR017" H 5400 1000 30  0001 C CNN
 F 1 "GND" H 5400 930 30  0001 C CNN
 F 2 "" H 5400 1000 60  0000 C CNN
@@
 MISO
 $Comp
-L VCC #PWR10
+L VCC #PWR018
 U 1 1 563EDBAF
 P 5400 700
-F 0 "#PWR10" H 5400 800 30  0001 C CNN
+F 0 "#PWR018" H 5400 800 30  0001 C CNN
 F 1 "VCC" H 5400 800 30  0000 C CNN
 F 2 "" H 5400 700 60  0000 C CNN
@@
 $EndComp
 $Comp
-L GND #PWR9
+L GND #PWR019
 U 1 1 563EFB35
 P 5350 2150
-F 0 "#PWR9" H 5350 2150 30  0001 C CNN
+F 0 "#PWR019" H 5350 2150 30  0001 C CNN
 F 1 "GND" H 5350 2080 30  0001 C CNN
 F 2 "" H 5350 2150 60  0000 C CNN
@@
 $EndComp
 $Comp
-L GND #PWR24
+L GND #PWR020
 U 1 1 563F09B8
 P 10750 2450
-F 0 "#PWR24" H 10750 2450 30  0001 C CNN
+F 0 "#PWR020" H 10750 2450 30  0001 C CNN
 F 1 "GND" H 10750 2380 30  0001 C CNN
 F 2 "" H 10750 2450 60  0000 C CNN
@@
 $EndComp
 $Comp
-L GND #PWR19
+L GND #PWR021
 U 1 1 563F123A
 P 8700 5600
-F 0 "#PWR19" H 8700 5600 30  0001 C CNN
+F 0 "#PWR021" H 8700 5600 30  0001 C CNN
 F 1 "GND" H 8700 5530 30  0001 C CNN
 F 2 "" H 8700 5600 60  0000 C CNN
@@
 $EndComp
 $Comp
-L GND #PWR18
+L GND #PWR022
 U 1 1 563F1826
 P 7800 5050
-F 0 "#PWR18" H 7800 5050 30  0001 C CNN
+F 0 "#PWR022" H 7800 5050 30  0001 C CNN
 F 1 "GND" H 7800 4980 30  0001 C CNN
 F 2 "" H 7800 5050 60  0000 C CNN
@@
 Text Label 7650 2650 3    60   ~ 0
 P9
-Text Label 4700 2550 2    60   ~ 0
-P2
 Text Label 4700 2650 2    60   ~ 0
-P3
+P4
 Text Label 4700 2750 2    60   ~ 0
-P4
+P5
 Text Label 4700 2850 2    60   ~ 0
-P5
+P6
 Text Label 4700 2950 2    60   ~ 0
-P6
-Text Label 4700 3050 2    60   ~ 0
 P8
 Text Label 7800 2650 3    60   ~ 0
@@
 Text Label 4700 3250 2    60   ~ 0
 P10
-Text Label 4700 3450 2    60   ~ 0
+Text Label 4450 2250 2    60   ~ 0
 P1
 $Comp
@@
 $EndComp
 $Comp
-L VDD #PWR5
+L VDD #PWR023
 U 1 1 563EF135
 P 3250 5000
-F 0 "#PWR5" H 3250 5100 30  0001 C CNN
+F 0 "#PWR023" H 3250 5100 30  0001 C CNN
 F 1 "VDD" H 3250 5110 30  0000 C CNN
 F 2 "" H 3250 5000 60  0000 C CNN
@@
 $EndComp
 $Comp
-L GND #PWR4
+L GND #PWR024
 U 1 1 563F26E5
 P 3000 6950
-F 0 "#PWR4" H 3000 6950 30  0001 C CNN
+F 0 "#PWR024" H 3000 6950 30  0001 C CNN
 F 1 "GND" H 3000 6880 30  0001 C CNN
 F 2 "" H 3000 6950 60  0000 C CNN
@@
 NoConn ~ 4300 1350
 NoConn ~ 4300 2050
-NoConn ~ 4300 2250
-NoConn ~ 4300 2350
 NoConn ~ 4300 4250
 $Comp
@@
 $EndComp
 $Comp
-L GND #PWR6
+L GND #PWR025
 U 1 1 5640122A
 P 3950 7700
-F 0 "#PWR6" H 3950 7700 30  0001 C CNN
+F 0 "#PWR025" H 3950 7700 30  0001 C CNN
 F 1 "GND" H 3950 7630 30  0001 C CNN
 F 2 "" H 3950 7700 60  0000 C CNN
@@
 $EndComp
 $Comp
-L GND #PWR13
+L GND #PWR026
 U 1 1 56401BCE
 P 6600 7350
-F 0 "#PWR13" H 6600 7350 30  0001 C CNN
+F 0 "#PWR026" H 6600 7350 30  0001 C CNN
 F 1 "GND" H 6600 7280 30  0001 C CNN
 F 2 "" H 6600 7350 60  0000 C CNN
@@
 	7800 2500 7800 2650
 Wire Wire Line
-	4700 2550 4300 2550
-Wire Wire Line
 	4300 2650 4700 2650
 Wire Wire Line
@@
 	4300 2950 4700 2950
 Wire Wire Line
-	4300 3050 4700 3050
-Wire Wire Line
 	4300 3150 4700 3150
 Wire Wire Line
 	4300 3250 4700 3250
-Wire Wire Line
-	4300 3450 4700 3450
 Wire Wire Line
 	1150 5500 1150 5600
@@
 Wire Wire Line
 	8250 6100 8500 6100
+$Sheet
+S -4400 850  2700 2600
+U 56646F09
+F0 "LCD_board" 50
+F1 "LCD_board.sch" 50
+$EndSheet
+Wire Wire Line
+	4300 2250 4450 2250
+Wire Wire Line
+	4300 2550 4700 2550
+Text Label 4700 2550 2    60   ~ 0
+P3
+NoConn ~ 4300 3050
+Wire Wire Line
+	4300 2350 4450 2350
+Text Label 4450 2350 2    60   ~ 0
+P2
+$Comp
+L GND #PWR027
+U 1 1 567B7B30
+P 5000 3400
+F 0 "#PWR027" H 5000 3400 30  0001 C CNN
+F 1 "GND" H 5000 3330 30  0001 C CNN
+F 2 "" H 5000 3400 60  0000 C CNN
+F 3 "" H 5000 3400 60  0000 C CNN
+	1    5000 3400
+	1    0    0    -1
+$EndComp
+$Comp
+L R R24
+U 1 1 567B7CBE
+P 4600 3350
+F 0 "R24" V 4680 3350 40  0000 C CNN
+F 1 "10K" V 4607 3351 40  0000 C CNN
+F 2 "~" V 4530 3350 30  0000 C CNN
+F 3 "~" H 4600 3350 30  0000 C CNN
+	1    4600 3350
+	0    1    1    0
+$EndComp
+Wire Wire Line
+	4300 3450 4300 3350
+Wire Wire Line
+	4300 3350 4350 3350
+Wire Wire Line
+	4850 3350 5000 3350
+Wire Wire Line
+	5000 3350 5000 3400
 $EndSCHEMATC

Commit message: Swapped EPIT1_EPIT0 with GPT_CMPOUT3. Fixed usb d+ d- switch issue.
Changed lines of the file:
@@
 Sheet 1 2
 Title ""
-Date "6 mar 2016"
+Date "12 aug 2016"
 Rev ""
 Comp ""
@@
 Text Label 6300 4750 2    60   ~ 0
 5V_DELAYED
-Text Label 3250 7400 0    60   ~ 0
+Text Label 6300 5800 3    60   ~ 0
 GPT_CMPOUT3
 NoConn ~ 4300 1350
@@
 Text Label 2400 7250 0    60   ~ 0
 5V_DELAYED
-Text Label 6300 5800 3    60   ~ 0
+Text Label 3250 7400 0    60   ~ 0
 EPIT1_EPIT0
 $Comp

Commit message: Added 5V breakout to kbrd panel. Changed BOM to reflect proper i2c (vs spi) encrypted eeprom chip. Made gerber files for kbrd only.
Parts:
- added P1: CPU_FAN, ~, symbol CONN_2
Connections:
- wire segments 333 -> 336
Changed lines of the file:
@@
 Sheet 1 2
 Title ""
-Date "12 aug 2016"
+Date "15 aug 2016"
 Rev ""
 Comp ""
@@
 Wire Wire Line
 	5000 3350 5000 3400
+$Comp
+L CONN_2 P1
+U 1 1 57B201A1
+P 4350 4650
+F 0 "P1" V 4300 4650 40  0000 C CNN
+F 1 "CPU_FAN" V 4400 4650 40  0000 C CNN
+F 2 "~" H 4350 4650 60  0000 C CNN
+F 3 "~" H 4350 4650 60  0000 C CNN
+	1    4350 4650
+	-1   0    0    1
+$EndComp
+Wire Wire Line
+	4700 4550 5100 4550
+Wire Wire Line
+	4700 4750 5100 4750
+$Comp
+L VDD #PWR028
+U 1 1 57B20564
+P 5100 4550
+F 0 "#PWR028" H 5100 4650 30  0001 C CNN
+F 1 "VDD" H 5100 4660 30  0000 C CNN
+F 2 "" H 5100 4550 60  0000 C CNN
+F 3 "" H 5100 4550 60  0000 C CNN
+	1    5100 4550
+	1    0    0    -1
+$EndComp
+$Comp
+L GND #PWR029
+U 1 1 57B2056A
+P 5100 4800
+F 0 "#PWR029" H 5100 4800 30  0001 C CNN
+F 1 "GND" H 5100 4730 30  0001 C CNN
+F 2 "" H 5100 4800 60  0000 C CNN
+F 3 "" H 5100 4800 60  0000 C CNN
+	1    5100 4800
+	1    0    0    -1
+$EndComp
+Wire Wire Line
+	5100 4750 5100 4800
 $EndSCHEMATC

Commit message: Adding LVDS 50 pin header to LCD front panel board. Also redoing reset pin for tusb2046b and crypto chip using RC circuit.
Connections:
- no-connect marks 14 -> 21
Changed lines of the file:
@@
 Sheet 1 2
 Title ""
-Date "15 aug 2016"
+Date "28 jan 2018"
 Rev ""
 Comp ""
@@
 Wire Wire Line
 	5100 4750 5100 4800
+NoConn ~ 7100 4950
+NoConn ~ 7650 6300
+NoConn ~ 7650 6100
+NoConn ~ 7900 5550
+NoConn ~ 8500 5350
+NoConn ~ 700  2800
+NoConn ~ 700  3000
 $EndSCHEMATC
