File: LCD_board.sch (KiCad schematic (older format))
At the start: 56 parts, among them CON2 AVR-ISP-6-DR, CON3 AVR-ISP-6-DR, Q10 MOSFET_N, Q11 MOSFET_N, Q9 MOSFET_N, SW5 MCU_RST, SW6 MCU_RST, SW7 SPST, U10 NHD-0440AZ-FL-YBW, U11 NRF24L01+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

Commit message: Adding LVDS 50 pin header to LCD front panel board. Also redoing reset pin for tusb2046b and crypto chip using RC circuit.
Parts:
- removed U15: MAX6749, symbol MAX6749
- removed U18: LVDS_HEADER, symbol LVDS_HEADER
- added C25, C26, C27, C28, C29, C30, C31, C32, C33, C34: 22pF, ~, symbol C
- added R39, R40, R42, R43, R44, R45, R46, R47, R48, R49: 27, ~, symbol R
- added R41: 10K, ~, symbol R
- added U15: PIXEL_QI_IPEX_BREAKOUT, symbol PIXEL_QI_IPEX_BREAKOUT
- added U18: LCD_50PIN, symbol LCD_50PIN
- C19: value 100pF -> 1uF
- R32: value 500K -> 15K
- R34: value 500K -> 1.5K
Connections:
- net labels added: OVCR
- wire segments 310 -> 362
- no-connect marks 44 -> 66
Other:
- moved on the sheet: C24, Q10, Q11, R37, R38, SW7, U10, U11

Commit message: 50 pin FFC cable now goes from motherboard to LCD board.
Parts:
- removed U15: PIXEL_QI_IPEX_BREAKOUT, symbol PIXEL_QI_IPEX_BREAKOUT
- removed U18: LCD_50PIN, symbol LCD_50PIN
Connections:
- wire segments 362 -> 328
- no-connect marks 66 -> 48
Other:
- moved on the sheet: C25, C26, C27, C28, C29, C30, C31, C32, C33, C34, R46, R47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
